File: LinkMeBaby.kicad_pcb (KiCad board)
At the start: 2 copper layers, 30.1 x 82.4 mm, 50 parts, among them J1 USB_C_Receptacle_USB2.0, J2 TEST_CONN, J3 GBC, J4 GBA, J5 TC2030-IDC-NL, U1 SN74LVC4245APWR, U2 USBLC6-2SC6, U3 STM32F407VET6, U4 MP2359DJ-LF-Z, Y1 16mhz

Commit message: LCSC part number hunting
Parts:
- D5, D6: value B5819W -> 1N5819HW-7-F
- U4: value MP2359DJ-LF-Z -> LMR14006YDDCR
Connections:
- J1 pad A8: (no net) -> Net-(J1-PadA8)
- J1 pad B8: (no net) -> Net-(J1-PadB8)
- J3 pad 4: (no net) -> Net-(J3-Pad4)
- U1 pad 10: (no net) -> Net-(U1-Pad10)
- U1 pad 14: (no net) -> Net-(U1-Pad14)
- U1 pad 15: (no net) -> Net-(U1-Pad15)
- U1 pad 16: (no net) -> Net-(U1-Pad16)
- U1 pad 17: (no net) -> Net-(U1-Pad17)
- U1 pad 7: (no net) -> Net-(U1-Pad7)
- U1 pad 8: (no net) -> Net-(U1-Pad8)
- U1 pad 9: (no net) -> Net-(U1-Pad9)
- U3 pad 1: (no net) -> Net-(U3-Pad1)
- U3 pad 15: (no net) -> Net-(U3-Pad15)
- U3 pad 16: (no net) -> Net-(U3-Pad16)
- U3 pad 17: (no net) -> Net-(U3-Pad17)
- U3 pad 18: (no net) -> Net-(U3-Pad18)
- U3 pad 2: (no net) -> Net-(U3-Pad2)
- U3 pad 21: (no net) -> Net-(U3-Pad21)
- U3 pad 23: (no net) -> Net-(U3-Pad23)
- U3 pad 24: (no net) -> Net-(U3-Pad24)
- U3 pad 25: (no net) -> Net-(U3-Pad25)
- U3 pad 26: (no net) -> Net-(U3-Pad26)
- U3 pad 3: (no net) -> Net-(U3-Pad3)
- U3 pad 34: (no net) -> Net-(U3-Pad34)
- U3 pad 35: (no net) -> Net-(U3-Pad35)
- U3 pad 36: (no net) -> Net-(U3-Pad36)
- U3 pad 37: (no net) -> Net-(U3-Pad37)
- U3 pad 38: (no net) -> Net-(U3-Pad38)
- U3 pad 39: (no net) -> Net-(U3-Pad39)
- U3 pad 4: (no net) -> Net-(U3-Pad4)
- U3 pad 40: (no net) -> Net-(U3-Pad40)
- U3 pad 41: (no net) -> Net-(U3-Pad41)
- U3 pad 42: (no net) -> Net-(U3-Pad42)
- U3 pad 43: (no net) -> Net-(U3-Pad43)
- U3 pad 44: (no net) -> Net-(U3-Pad44)
- U3 pad 45: (no net) -> Net-(U3-Pad45)
- U3 pad 46: (no net) -> Net-(U3-Pad46)
- U3 pad 47: (no net) -> Net-(U3-Pad47)
- U3 pad 48: (no net) -> Net-(U3-Pad48)
- U3 pad 5: (no net) -> Net-(U3-Pad5)
- U3 pad 51: (no net) -> Net-(U3-Pad51)
- U3 pad 52: (no net) -> Net-(U3-Pad52)
- U3 pad 53: (no net) -> Net-(U3-Pad53)
- U3 pad 54: (no net) -> Net-(U3-Pad54)
- U3 pad 55: (no net) -> Net-(U3-Pad55)
- U3 pad 56: (no net) -> Net-(U3-Pad56)
- U3 pad 57: (no net) -> Net-(U3-Pad57)
- U3 pad 58: (no net) -> Net-(U3-Pad58)
- U3 pad 59: (no net) -> Net-(U3-Pad59)
- U3 pad 60: (no net) -> Net-(U3-Pad60)
- U3 pad 61: (no net) -> Net-(U3-Pad61)
- U3 pad 62: (no net) -> Net-(U3-Pad62)
- U3 pad 63: (no net) -> Net-(U3-Pad63)
- U3 pad 64: (no net) -> Net-(U3-Pad64)
- U3 pad 65: (no net) -> Net-(U3-Pad65)
- U3 pad 66: (no net) -> Net-(U3-Pad66)
- U3 pad 67: (no net) -> Net-(U3-Pad67)
- U3 pad 68: (no net) -> Net-(U3-Pad68)
- U3 pad 69: (no net) -> Net-(U3-Pad69)
- U3 pad 7: (no net) -> Net-(U3-Pad7)
- U3 pad 77: (no net) -> Net-(U3-Pad77)
- U3 pad 78: (no net) -> Net-(U3-Pad78)
- U3 pad 79: (no net) -> Net-(U3-Pad79)
- U3 pad 8: (no net) -> Net-(U3-Pad8)
- U3 pad 80: (no net) -> Net-(U3-Pad80)
- U3 pad 81: (no net) -> Net-(U3-Pad81)
- U3 pad 82: (no net) -> Net-(U3-Pad82)
- U3 pad 83: (no net) -> Net-(U3-Pad83)
- U3 pad 84: (no net) -> Net-(U3-Pad84)
- U3 pad 85: (no net) -> Net-(U3-Pad85)
- U3 pad 86: (no net) -> Net-(U3-Pad86)
- U3 pad 87: (no net) -> Net-(U3-Pad87)
- U3 pad 88: (no net) -> Net-(U3-Pad88)
- U3 pad 9: (no net) -> Net-(U3-Pad9)
- U3 pad 95: (no net) -> Net-(U3-Pad95)
- U3 pad 96: (no net) -> Net-(U3-Pad96)
- U3 pad 97: (no net) -> Net-(U3-Pad97)
- U3 pad 98: (no net) -> Net-(U3-Pad98)

Commit message: lol redo the entire thing
Parts:
- removed C13, C14, C15: 100n, Capacitor_SMD:C_0402_1005Metric_Pad0.74x0.62mm_HandSolder
- U3: value STM32F407VET6 -> STM32F401CBUx; footprint Package_QFP:LQFP-100_14x14mm_P0.5mm -> Package_DFN_QFN:QFN-48-1EP_7x7mm_P0.5mm_EP5.6x5.6mm
- moved R14 35.5 mm to (21.9, 75.0), turned to 180 degrees
- moved D7 33.8 mm to (25.4, 75.0), turned to 0 degrees
- moved R3 27.3 mm to (21.9, 69.7), turned to 0 degrees
- moved R4 26.4 mm to (21.9, 71.5), turned to 0 degrees
- moved R7 26.4 mm to (21.9, 68.0), turned to 0 degrees
- moved R6 26.0 mm to (21.9, 73.2), turned to 0 degrees
- moved C2 24.9 mm to (40.1, 60.5), turned to 180 degrees
- moved J5 23.7 mm to (25.3, 82.8), turned to 270 degrees
- moved C6 21.9 mm to (45.1, 70.1), turned to 180 degrees
- moved D1 20.8 mm to (25.4, 69.7), turned to 0 degrees
- moved C1 20.1 mm to (36.9, 67.2)
- moved D2 19.6 mm to (25.4, 71.5), turned to 0 degrees
- moved D4 19.6 mm to (25.4, 68.0), turned to 0 degrees
- moved C11 19.1 mm to (36.7, 69.2)
- moved D3 19.0 mm to (25.4, 73.2), turned to 0 degrees
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Connections:
- J1 pad A8: Net-(J1-PadA8) -> (no net)
- J1 pad B8: Net-(J1-PadB8) -> (no net)
- J3 pad 4: Net-(J3-Pad4) -> (no net)
- U1 pad 10: Net-(U1-Pad10) -> (no net)
- U1 pad 14: Net-(U1-Pad14) -> (no net)
- U1 pad 15: Net-(U1-Pad15) -> (no net)
- U1 pad 16: Net-(U1-Pad16) -> (no net)
- U1 pad 17: Net-(U1-Pad17) -> (no net)
- U1 pad 7: Net-(U1-Pad7) -> (no net)
- U1 pad 8: Net-(U1-Pad8) -> (no net)
- U1 pad 9: Net-(U1-Pad9) -> (no net)
- U3 pad 1: Net-(U3-Pad1) -> +3V3
- U3 pad 10: GND -> (no net)
- U3 pad 11: +3V3 -> (no net)
- U3 pad 12: HSE_IN -> (no net)
- U3 pad 13: HSE_OUT -> DIR
- U3 pad 14: NRST -> SPI1_NSS
- U3 pad 15: Net-(U3-Pad15) -> SPI1_SCK
- U3 pad 16: Net-(U3-Pad16) -> SPI1_MISO
- U3 pad 17: Net-(U3-Pad17) -> SPI1_MOSI
- U3 pad 18: Net-(U3-Pad18) -> STATUS_SD
- U3 pad 19: +3V3 -> STATUS_CK
- U3 pad 2: Net-(U3-Pad2) -> (no net)
- U3 pad 20: GND -> STATUS_SO
- U3 pad 21: Net-(U3-Pad21) -> STATUS_SI
- U3 pad 22: +3V3 -> Net-(C1-Pad1)
- U3 pad 23: Net-(U3-Pad23) -> GND
- U3 pad 24: Net-(U3-Pad24) -> +3V3
- U3 pad 25: Net-(U3-Pad25) -> (no net)
- U3 pad 26: Net-(U3-Pad26) -> (no net)
- U3 pad 27: GND -> (no net)
- U3 pad 28: +3V3 -> (no net)
- U3 pad 29: SPI1_NSS -> (no net)
- U3 pad 3: Net-(U3-Pad3) -> (no net)
- U3 pad 30: SPI1_SCK -> (no net)
- U3 pad 31: SPI1_MISO -> (no net)
- U3 pad 32: SPI1_MOSI -> USB_D-
- U3 pad 33: DIR -> USB_D+
- U3 pad 34: Net-(U3-Pad34) -> SWDIO
- U3 pad 35: Net-(U3-Pad35) -> GND
- U3 pad 36: Net-(U3-Pad36) -> +3V3
- U3 pad 37: Net-(U3-Pad37) -> SWCLK
- U3 pad 38: Net-(U3-Pad38) -> (no net)
- U3 pad 39: Net-(U3-Pad39) -> SWO
- U3 pad 4: Net-(U3-Pad4) -> (no net)
- U3 pad 40: Net-(U3-Pad40) -> (no net)
- U3 pad 41: Net-(U3-Pad41) -> (no net)
- U3 pad 42: Net-(U3-Pad42) -> (no net)
- U3 pad 43: Net-(U3-Pad43) -> (no net)
- U3 pad 44: Net-(U3-Pad44) -> Net-(R5-Pad1)
- U3 pad 45: Net-(U3-Pad45) -> (no net)
- U3 pad 46: Net-(U3-Pad46) -> (no net)
- U3 pad 47: Net-(U3-Pad47) -> GND
- U3 pad 48: Net-(U3-Pad48) -> +3V3
- U3 pad 49: Net-(C1-Pad1) -> GND
- U3 pad 5: Net-(U3-Pad5) -> HSE_IN
- U3 pad 6: +3V3 -> HSE_OUT
- U3 pad 7: Net-(U3-Pad7) -> NRST
- U3 pad 8: Net-(U3-Pad8) -> GND
- U3 pad 9: Net-(U3-Pad9) -> Net-(C2-Pad1)
Routing:
- net +3V3: track 93.0 -> 70.9 mm, vias 16 -> 14
- net SWCLK: track 52.9 -> 31.9 mm
- net SWO: track 55.3 -> 35.4 mm
- net STATUS_SI: track 4.26 -> 15.1 mm
- net SWDIO: track 39.7 -> 29.0 mm
- net STATUS_SD: track 3.02 -> 13.6 mm
- net STATUS_SO: track 4.63 -> 14.8 mm
- net DIR: track 29.7 -> 21.0 mm
- net STATUS_CK: track 5.79 -> 14.0 mm
- net NRST: track 52.3 -> 44.1 mm, vias 2 -> 4
- net Net-(D5-Pad1): track 8.79 -> 2.36 mm
- net BUCK_IN: track 17.1 -> 11.2 mm
- net +5V: track 26.6 -> 32.4 mm
- net BUCK_SW: track 11.8 -> 5.98 mm
- net GND: track 167.4 -> 163.1 mm, vias 33 -> 26
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Other:
- board size 30.1 x 82.4 mm -> 30.1 x 70.4 mm
