File: LinkMeBaby.sch (KiCad schematic (older format))
At the start: 50 parts, among them J1 USB_C_Receptacle_USB2.0, J2 TEST_CONN, J3 GBC, J4 GBA, J5 TC2030-IDC-NL, U1 SN74LVC4245APWR, U2 USBLC6-2SC6, U3 STM32F407VET6, U4 MP2359DJ-LF-Z, Y1 16mhz

Commit message: LCSC part number hunting
Parts:
- C1, C10, C11, C12, C13, C14, C15, C16, C2, C3, C4, C5, C6, C7, C8, C9: symbol Device:C_Small -> LinkMeBaby-rescue:C_Small-Device
- D1, D2, D3, D4: symbol Device:LED_Small -> LinkMeBaby-rescue:LED_Small-Device; LCSC_PN C2286 -> C72041
- D5, D6: value B5819W -> 1N5819HW-7-F; symbol Device:D_Schottky_Small -> LinkMeBaby-rescue:D_Schottky_Small-Device; LCSC_PN C8598 -> C82544
- D7: symbol Device:LED_Small -> LinkMeBaby-rescue:LED_Small-Device; LCSC_PN C2286 -> C72044
- F1: symbol Device:Polyfuse_Small -> LinkMeBaby-rescue:Polyfuse_Small-Device
- FB1: symbol Device:Ferrite_Bead_Small -> LinkMeBaby-rescue:Ferrite_Bead_Small-Device
- J1: symbol Connector:USB_C_Receptacle_USB2.0 -> LinkMeBaby-rescue:USB_C_Receptacle_USB2.0-Connector
- J2: symbol Connector:Conn_01x06_Female -> LinkMeBaby-rescue:Conn_01x06_Female-Connector
- L1: symbol Device:L_Small -> LinkMeBaby-rescue:L_Small-Device
- R1, R10, R11, R12, R13, R14, R2, R5, R8, R9: symbol Device:R_Small -> LinkMeBaby-rescue:R_Small-Device
- R3, R4, R6, R7: symbol Device:R_Small -> LinkMeBaby-rescue:R_Small-Device; LCSC_PN C22843 -> C25989
- U1: symbol SN74LVC4245APWR:SN74LVC4245APWR -> LinkMeBaby-rescue:SN74LVC4245APWR-SN74LVC4245APWR
- U2: symbol Power_Protection:USBLC6-2SC6 -> LinkMeBaby-rescue:USBLC6-2SC6-Power_Protection
- U3: symbol MCU_ST_STM32F4:STM32F407VETx -> LinkMeBaby-rescue:STM32F407VETx-MCU_ST_STM32F4
- U4: value MP2359DJ-LF-Z -> LMR14006YDDCR; LCSC_PN C14259 -> C477919
- Y1: symbol Device:Crystal_GND24_Small -> LinkMeBaby-rescue:Crystal_GND24_Small-Device

Commit message: lol redo the entire thing
Parts:
- removed C13, C14, C15: 100n, Capacitor_SMD:C_0402_1005Metric_Pad0.74x0.62mm_HandSolder, symbol LinkMeBaby-rescue:C_Small-Device
- removed U3: STM32F407VET6, Package_QFP:LQFP-100_14x14mm_P0.5mm, symbol LinkMeBaby-rescue:STM32F407VETx-MCU_ST_STM32F4
- added U3: STM32F401CBUx, Package_DFN_QFN:QFN-48-1EP_7x7mm_P0.5mm_EP5.6x5.6mm, symbol STM:STM32F401CBUx
Connections:
- net +3V3: now also U3.1 (VBAT), U3.24 (VDD), U3.36 (VDD), U3.48 (VDD)
- net DIR: now also U3.13 (PA3)
- net GND: now also U3.23 (VSS), U3.35 (VSS), U3.47 (VSS), U3.49 (VSS), U3.8 (VSSA)
- net HSE_IN: now also U3.5 (PH0)
- net HSE_OUT: now also U3.6 (PH1)
- net NRST: now also U3.7 (NRST)
- net SPI1_MISO: now also U3.16 (PA6)
- net SPI1_MOSI: now also U3.17 (PA7)
- net SPI1_NSS: now also U3.14 (PA4)
- net SPI1_SCK: now also U3.15 (PA5)
- net STATUS_CK: now also U3.19 (PB1)
- net STATUS_SD: now also U3.18 (PB0)
- net STATUS_SI: now also U3.21 (PB10)
- net STATUS_SO: now also U3.20 (PB2)
- net SWCLK: now also U3.37 (PA14)
- net SWDIO: now also U3.34 (PA13)
- net SWO: now also U3.39 (PB3)
- net USB_D+: now also U3.33 (PA12)
- net USB_D-: now also U3.32 (PA11)
- net at C1.1: now also U3.22 (VCAP1)
- net at C2.1: now also U3.9 (VREF+)
- net at R5.1: now also U3.44 (BOOT0)
- no-connect marks 77 -> 12
Other:
- moved on the sheet: C1, C2, R5, U2
