File: hardware/LinkMeBaby.kicad_pcb (KiCad board)
At the start: 2 copper layers, 30.1 x 70.4 mm, 47 parts, among them J1 USB_C_Receptacle_USB2.0, J2 TEST_CONN, J3 GBC, J4 GBA, J5 TC2030-IDC-NL, U1 SN74LVC4245APWR, U2 USBLC6-2SC6, U3 STM32F401CBUx, U4 LMR14006YDDCR, Y1 16mhz

Commit message: Getting close...
Parts:
- added C13: 100n, Capacitor_SMD:C_0402_1005Metric_Pad0.74x0.62mm_HandSolder, F.Cu at (33.5, 59.0)
- added R15: 4k7, Resistor_SMD:R_0402_1005Metric_Pad0.72x0.64mm_HandSolder, F.Cu at (48.6, 66.3)
- added R16: 4k7, Resistor_SMD:R_0402_1005Metric_Pad0.72x0.64mm_HandSolder, F.Cu at (48.6, 65.2)
- added U5: ATECC608A-SSHDA-B, Package_SO:SOIC-8_3.9x4.9mm_P1.27mm, F.Cu at (33.5, 55.6)
- Y1: value 16mhz -> 25mhz
- moved R5 2.94 mm to (48.4, 61.7), turned to 90 degrees
- moved C3 1.71 mm to (36.7, 69.8)
- moved C4 1.52 mm to (47.0, 61.1), turned to 90 degrees
- moved C11 0.70 mm to (36.7, 68.5)
- renumbered J4 to GBA, J3 to GBC
Connections:
- U3 pad 42: (no net) -> I2C1_SCL
- U3 pad 43: (no net) -> I2C1_SDA
Routing:
- net I2C1_SCL: track 0.00 -> 20.8 mm, vias 0 -> 2
- net I2C1_SDA: track 0.00 -> 17.9 mm, vias 0 -> 2
- net +3V3: track 70.9 -> 88.1 mm, vias 14 -> 17
- net Net-(R5-Pad1): track 1.51 -> 4.24 mm
- net GND: track 163.1 -> 161.2 mm, vias 26 -> 24
- net DIR: track 21.0 -> 21.7 mm
Other:
- outline, holes or cut-outs redrawn
- board text added: "GBA USB Adapter v0.1.0"
- board text added: "GND"
- board text added: "SC"
- board text added: "SD"
- board text added: "SI"
- board text added: "SO"
- board text added: "VDD"
- board text added: "| GND | SD | SO |"
- board text added: "| SC | VDD | SI |"
