File: hardware/LinkMeBaby.sch (KiCad schematic (older format))
At the start: 47 parts, among them J1 USB_C_Receptacle_USB2.0, J2 TEST_CONN, J3 GBC, J4 GBA, J5 TC2030-IDC-NL, U1 SN74LVC4245APWR, U2 USBLC6-2SC6, U3 STM32F401CBUx, U4 LMR14006YDDCR, Y1 16mhz

Commit message: Getting close...
Parts:
- added C13: 100n, Capacitor_SMD:C_0402_1005Metric_Pad0.74x0.62mm_HandSolder, symbol LinkMeBaby-rescue:C_Small-Device
- added R15, R16: 4k7, Resistor_SMD:R_0402_1005Metric_Pad0.72x0.64mm_HandSolder, symbol Device:R_Small
- added U5: ATECC608A-SSHDA-B, Package_SO:SOIC-8_3.9x4.9mm_P1.27mm, symbol Security:ATECC608A-SSHDA
- Y1: value 16mhz -> 25mhz; LCSC_PN C13738 -> C439049
Connections:
- net +3V3: now also C13.1, R15.1, R16.1, U5.8 (VCC)
- net GND: now also C13.2, U5.4 (GND)
- net I2C1_SCL: now reaches U3.42 (PB6)
- net I2C1_SCL: now also R15.2, U5.6 (SCL)
- net I2C1_SDA: now reaches U3.43 (PB7)
- net I2C1_SDA: now also R16.2, U5.5 (SDA)
Changed lines of the file:
@@
 P 9000 5850
 F 0 "Y1" H 8850 6000 50  0000 L CNN
-F 1 "16mhz" H 8750 6100 50  0000 L CNN
+F 1 "25mhz" H 8750 6100 50  0000 L CNN
 F 2 "Crystal:Crystal_SMD_3225-4Pin_3.2x2.5mm" H 9000 5850 50  0001 C CNN
-F 3 "https://datasheet.lcsc.com/szlcsc/Yangxing-Tech-X322516MLB4SI_C13738.pdf" H 9000 5850 50  0001 C CNN
-F 4 "C13738" H 9000 5850 50  0001 C CNN "LCSC_PN"
+F 3 "https://datasheet.lcsc.com/lcsc/1912111437_Shenzhen-SCTF-Elec-S3B25-000000F1010F30_C439049.pdf" H 9000 5850 50  0001 C CNN
+F 4 "C439049" H 9000 5850 50  0001 C CNN "LCSC_PN"
 F 5 "SMD-CRY-3225_4P" H 9000 5850 50  0001 C CNN "LCSC_FP"
 	1    9000 5850
@@
 	5600 4300 5600 4400
 Connection ~ 5600 4400
+$Comp
+L Security:ATECC608A-SSHDA U5
+U 1 1 609D73D1
+P 5750 5600
+F 0 "U5" H 5900 5850 50  0000 R CNN
+F 1 "ATECC608A-SSHDA-B" H 6650 5300 50  0000 R CNN
+F 2 "Package_SO:SOIC-8_3.9x4.9mm_P1.27mm" H 5750 5600 50  0001 C CNN
+F 3 "https://datasheet.lcsc.com/lcsc/1912111437_Microchip-Tech-ATECC608A-SSHDA-B_C376619.pdf" H 5900 5850 50  0001 C CNN
+F 4 "C376619" H 5750 5600 50  0001 C CNN "LCSC_PN"
+F 5 "SOIC-8" H 5750 5600 50  0001 C CNN "LCSC_FP"
+	1    5750 5600
+	1    0    0    -1
+$EndComp
+$Comp
+L LinkMeBaby-rescue:C_Small-Device C13
+U 1 1 609EFDE1
+P 5200 5600
+F 0 "C13" H 5292 5646 50  0000 L CNN
+F 1 "100n" H 5292 5555 50  0000 L CNN
+F 2 "Capacitor_SMD:C_0402_1005Metric_Pad0.74x0.62mm_HandSolder" H 5200 5600 50  0001 C CNN
+F 3 "https://datasheet.lcsc.com/lcsc/1810191219_Samsung-Electro-Mechanics-CL05B104KO5NNNC_C1525.pdf" H 5200 5600 50  0001 C CNN
+F 4 "C1525" H 5200 5600 50  0001 C CNN "LCSC_PN"
+F 5 "0402" H 5200 5600 50  0001 C CNN "LCSC_FP"
+	1    5200 5600
+	1    0    0    -1
+$EndComp
+$Comp
+L LinkMeBaby-rescue:GND-power #PWR?
+U 1 1 609F62FB
+P 5750 5900
+F 0 "#PWR?" H 5750 5650 50  0001 C CNN
+F 1 "GND" H 5755 5727 50  0000 C CNN
+F 2 "" H 5750 5900 50  0001 C CNN
+F 3 "" H 5750 5900 50  0001 C CNN
+	1    5750 5900
+	1    0    0    -1
+$EndComp
+$Comp
+L LinkMeBaby-rescue:+3.3V-power #PWR?
+U 1 1 609F68F1
+P 5750 5300
+F 0 "#PWR?" H 5750 5150 50  0001 C CNN
+F 1 "+3.3V" H 5765 5473 50  0000 C CNN
+F 2 "" H 5750 5300 50  0001 C CNN
+F 3 "" H 5750 5300 50  0001 C CNN
+	1    5750 5300
+	1    0    0    -1
+$EndComp
+$Comp
+L LinkMeBaby-rescue:+3.3V-power #PWR?
+U 1 1 609F6F78
+P 5200 5500
+F 0 "#PWR?" H 5200 5350 50  0001 C CNN
+F 1 "+3.3V" H 5215 5673 50  0000 C CNN
+F 2 "" H 5200 5500 50  0001 C CNN
+F 3 "" H 5200 5500 50  0001 C CNN
+	1    5200 5500
+	1    0    0    -1
+$EndComp
+$Comp
+L LinkMeBaby-rescue:GND-power #PWR?
+U 1 1 609F75D3
+P 5200 5700
+F 0 "#PWR?" H 5200 5450 50  0001 C CNN
+F 1 "GND" H 5205 5527 50  0000 C CNN
+F 2 "" H 5200 5700 50  0001 C CNN
+F 3 "" H 5200 5700 50  0001 C CNN
+	1    5200 5700
+	1    0    0    -1
+$EndComp
+Text GLabel 4800 3400 0    50   Input ~ 0
+I2C1_SDA
+Text GLabel 4800 3300 0    50   Input ~ 0
+I2C1_SCL
+Text GLabel 6050 5700 2    50   Input ~ 0
+I2C1_SCL
+Text GLabel 6050 5500 2    50   Input ~ 0
+I2C1_SDA
+Text GLabel 7050 5700 3    50   Input ~ 0
+I2C1_SDA
+Text GLabel 6800 5700 3    50   Input ~ 0
+I2C1_SCL
+$Comp
+L Device:R_Small R15
+U 1 1 60A281DE
+P 6800 5600
+F 0 "R15" H 6859 5646 50  0000 L CNN
+F 1 "4k7" H 6859 5555 50  0000 L CNN
+F 2 "Resistor_SMD:R_0402_1005Metric_Pad0.72x0.64mm_HandSolder" H 6800 5600 50  0001 C CNN
+F 3 "https://datasheet.lcsc.com/lcsc/1810170731_TA-I-Tech-RMS04JT472_C208992.pdf" H 6800 5600 50  0001 C CNN
+F 4 "C208992" H 6800 5600 50  0001 C CNN "LCSC_PN"
+F 5 "0402" H 6800 5600 50  0001 C CNN "LCSC_FP"
+	1    6800 5600
+	1    0    0    -1
+$EndComp
+$Comp
+L Device:R_Small R16
+U 1 1 60A29FD4
+P 7050 5600
+F 0 "R16" H 7109 5646 50  0000 L CNN
+F 1 "4k7" H 7109 5555 50  0000 L CNN
+F 2 "Resistor_SMD:R_0402_1005Metric_Pad0.72x0.64mm_HandSolder" H 7050 5600 50  0001 C CNN
+F 3 "https://datasheet.lcsc.com/lcsc/1810170731_TA-I-Tech-RMS04JT472_C208992.pdf" H 7050 5600 50  0001 C CNN
+F 4 "C208992" H 7050 5600 50  0001 C CNN "LCSC_PN"
+F 5 "0402" H 7050 5600 50  0001 C CNN "LCSC_FP"
+	1    7050 5600
+	1    0    0    -1
+$EndComp
+$Comp
+L LinkMeBaby-rescue:+3.3V-power #PWR?
+U 1 1 60A3742A
+P 6800 5300
+F 0 "#PWR?" H 6800 5150 50  0001 C CNN
+F 1 "+3.3V" H 6815 5473 50  0000 C CNN
+F 2 "" H 6800 5300 50  0001 C CNN
+F 3 "" H 6800 5300 50  0001 C CNN
+	1    6800 5300
+	1    0    0    -1
+$EndComp
+Wire Wire Line
+	6800 5500 6800 5300
+$Comp
+L LinkMeBaby-rescue:+3.3V-power #PWR?
+U 1 1 60A3CFCF
+P 7050 5300
+F 0 "#PWR?" H 7050 5150 50  0001 C CNN
+F 1 "+3.3V" H 7065 5473 50  0000 C CNN
+F 2 "" H 7050 5300 50  0001 C CNN
+F 3 "" H 7050 5300 50  0001 C CNN
+	1    7050 5300
+	1    0    0    -1
+$EndComp
+Wire Wire Line
+	7050 5500 7050 5300
 $EndSCHEMATC
