File: hardware/cable-link.kicad_pcb (KiCad board)
At the start: 4 copper layers, 50 x 50 mm, 57 parts, among them J1 USB_C_Receptacle_USB2.0, J2 Conn_01x02, J3 GBA-LINK, Q1 BSS138, Q2 BSS138, Q3 BSS138, Q4 BSS138, U1 NCP1117-3.3_SOT223, U2 RP2040, U3 ATECC608A-MAHDA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

Commit message: Finish BOM
Parts:
- removed G***: LOGO, Connector_GBA:gba-logo
- removed G***: LOGO, Connector_GBA:opensourcehardware
- added J4: SWD, Connector_SWD:20021221-00010C4LF, F.Cu at (66.1, 48.8)
- C6: value 1u -> 2u2
- R4, R5: value 10k -> 470
- moved C5 7.41 mm to (56.3, 23.9), turned to 0 degrees
- moved C9 4.77 mm to (56.3, 27.0), turned to 0 degrees
Connections:
- U2 pad 24: (no net) -> /SWCLK
- U2 pad 25: (no net) -> /SWD
- U2 pad 26: (no net) -> +3V3
Routing:
- net +3V3: track 101.1 -> 104.5 mm

Commit message: Finish PCB layout
Parts:
- added G***: LOGO, Connector_GBA:gba-logo, B.Cu at (44.4, 45.0)
- added G***: LOGO, Connector_GBA:opensourcehardware, F.Cu at (32.5, 63.5)
- moved C5 7.38 mm to (56.1, 31.3), turned to 90 degrees
- moved C9 4.80 mm to (58.2, 31.4), turned to 90 degrees
- moved C4 2.99 mm to (52.5, 46.6)
- moved C13 0.30 mm to (49.1, 46.1)
Routing:
- net /SWCLK: track 0.00 -> 21.5 mm
- net /SWD: track 0.00 -> 20.4 mm
- net GND: track 88.6 -> 96.6 mm, vias 11 -> 13
- net +1V1: track 17.1 -> 20.6 mm
