File: hardware/cable-link.sch (KiCad schematic (older format))
At the start: 55 parts, among them J1 USB_C_Receptacle_USB2.0, J2 Conn_01x02, J3 GBA-LINK, Q1 BSS138, Q2 BSS138, Q3 BSS138, Q4 BSS138, U1 NCP1117-3.3_SOT223, U2 RP2040, U3 ATECC608A-MAHDA, U4 W25Q128JVS, Y1 12mhz

Commit message: Finish BOM
Parts:
- removed C5, C9: 10u, Capacitor_SMD:C_0805_2012Metric, symbol Device:C_Small
- added C5, C9: 10u, Capacitor_SMD:C_0805_2012Metric, symbol Device:CP_Small
- added J4: SWD, Connector_SWD:20021221-00010C4LF, symbol Connector:Conn_ARM_JTAG_SWD_10
- C1, C2: LCSC_FP (none) -> 0402; LCSC_PN (none) -> C387970; Manufacturer (none) -> Walsin Tech Corp; Mfg Part # (none) -> 0402N150G500CT
- C10, C12, C13, C14, C15, C16, C17, C18, C8: LCSC_FP (none) -> 0402; LCSC_PN (none) -> C541405; Manufacturer (none) -> YAGEO; Mfg Part # (none) -> CC0402KRX5R5BB104
- C11: LCSC_FP (none) -> 0805; LCSC_PN (none) -> C408141; Manufacturer (none) -> Murata Electronics; Mfg Part # (none) -> GRM21BR61C106KE15K
- C3, C4: LCSC_FP (none) -> 0603; LCSC_PN (none) -> C167641; Manufacturer (none) -> Vishay Intertech; Mfg Part # (none) -> VJ0603Y104JXACW1BC
- C6: value 1u -> 2u2; LCSC_FP (none) -> 0402; LCSC_PN (none) -> C193620; Manufacturer (none) -> FH(Guangdong Fenghua Advanced Tech); Mfg Part # (none) -> 0402X225K6R3NT
- C7: LCSC_FP (none) -> 0402; LCSC_PN (none) -> C193620; Manufacturer (none) -> FH(Guangdong Fenghua Advanced Tech); Mfg Part # (none) -> 0402X225K6R3NT
- D1, D2: LCSC_FP (none) -> SMD; LCSC_PN (none) -> C160479; Manufacturer (none) -> Lite-On; Mfg Part # (none) -> LTST-C281KGKT
- J1: LCSC_FP (none) -> 8.94*7.3mm; LCSC_PN (none) -> C165948; Manufacturer (none) -> Korean Hroparts Elec; Mfg Part # (none) -> TYPE-C-31-M-12
- J2: LCSC_FP (none) -> Through Hole,P=2.54mm; LCSC_PN (none) -> C358684; Manufacturer (none) -> MINTRON; Mfg Part # (none) -> MTP125-1102S1
- Q1, Q2, Q3, Q4: LCSC_FP (none) -> SOT-23(SOT-23-3); LCSC_PN (none) -> C193019; Manufacturer (none) -> AnBon; Mfg Part # (none) -> BSS138
- R1, R2, R3, R8: LCSC_FP (none) -> 0402; LCSC_PN (none) -> C226166; Manufacturer (none) -> FH(Guangdong Fenghua Advanced Tech); Mfg Part # (none) -> RC-02W1001FT
- R10, R11, R12, R13, R14, R15, R16, R17, R18, R19: LCSC_FP (none) -> 0402; LCSC_PN (none) -> C258091; Manufacturer (none) -> FH(Guangdong Fenghua Advanced Tech); Mfg Part # (none) -> RC-02W1002FT
- R4, R5: value 10k -> 470; LCSC_FP (none) -> 0603; LCSC_PN (none) -> C116694; Manufacturer (none) -> FH(Guangdong Fenghua Advanced Tech); Mfg Part # (none) -> RS-03K4700FT
- R6, R7: LCSC_FP (none) -> 0603; LCSC_PN (none) -> C321830; Manufacturer (none) -> FH(Guangdong Fenghua Advanced Tech); Mfg Part # (none) -> RS-03K27R0FT
- R9: LCSC_FP (none) -> 0402; LCSC_PN (none) -> C136582; Manufacturer (none) -> FH(Guangdong Fenghua Advanced Tech); Mfg Part # (none) -> RC-02000FT
- U1: LCSC_FP (none) -> SOT-223; LCSC_PN (none) -> C146799; Manufacturer (none) -> ON Semiconductor; Mfg Part # (none) -> NCP1117LPST33T3G
- U2: Manufacturer (none) -> Raspberry Pi; Mfg Part # (none) -> RP2040
- U3: LCSC_FP (none) -> UDFN-8; LCSC_PN (none) -> C616908; Manufacturer (none) -> Microchip Technology; Mfg Part # (none) -> ATECC608A-MAHDA-S
- U4: LCSC_FP (none) -> SOIC-8_208mil; LCSC_PN (none) -> C113767; Manufacturer (none) -> Winbond Elec; Mfg Part # (none) -> W25Q128JVSIQ
- Y1: LCSC_FP (none) -> SMD-3225_4P; LCSC_PN (none) -> C521582; Manufacturer (none) -> TAITIEN Elec; Mfg Part # (none) -> XXHCCLNANF-12.000000MHZ
Connections:
- net RUN is gone; now on net +3V3: U2.26 (RUN)
- net +3V3: now also C9.1
- net GND: now also C5.2, C9.2, J4.3 (GND), J4.5 (GND), J4.9 (GNDDetect)
- net SWCLK: now also J4.4 (SWDCLK/TCK)
- net SWD: now also J4.2 (SWDIO/TMS)
- net VBUS: now also C5.1
- no-connect marks 24 -> 28

Commit message: Finish PCB layout
Parts:
- C1, C2: Manufacturer Walsin Tech Corp -> Walsin Tech Corp
Changed lines of the file:
@@
 F 4 "0402" H 700 6150 50  0001 C CNN "LCSC_FP"
 F 5 "C387970" H 700 6150 50  0001 C CNN "LCSC_PN"
-F 6 " 	Walsin Tech Corp" H 700 6150 50  0001 C CNN "Manufacturer"
+F 6 "Walsin Tech Corp" H 700 6150 50  0001 C CNN "Manufacturer"
 F 7 "0402N150G500CT" H 700 6150 50  0001 C CNN "Mfg Part #"
 	1    700  6150
@@
 F 4 "0402" H 1400 6150 50  0001 C CNN "LCSC_FP"
 F 5 "C387970" H 1400 6150 50  0001 C CNN "LCSC_PN"
-F 6 " 	Walsin Tech Corp" H 1400 6150 50  0001 C CNN "Manufacturer"
+F 6 "Walsin Tech Corp" H 1400 6150 50  0001 C CNN "Manufacturer"
 F 7 "0402N150G500CT" H 1400 6150 50  0001 C CNN "Mfg Part #"
 	1    1400 6150

Commit message: Hardware Rev. C
Redesigned the board yet again. Order placed w/ JLCPCB.
Parts:
- removed C16, C17: 100n, Capacitor_SMD:C_0402_1005Metric, symbol Device:C_Small
- removed C5, C9: 10u, Capacitor_SMD:C_0805_2012Metric, symbol Device:CP_Small
- removed D1, D2: RED, LED_SMD:LED_0603_1608Metric, symbol Device:LED_Small
- removed J2: Conn_01x02, Connector_PinHeader_1.27mm:PinHeader_2x01_P1.27mm_Vertical_SMD, symbol Connector_Generic:Conn_01x02
- removed J3: GBA-LINK, Connector_GBA:GBA-LINK, symbol cable-link:GBA-LINK
- removed J4: SWD, Connector_SWD:20021221-00010C4LF, symbol Connector:Conn_ARM_JTAG_SWD_10
- removed Q1, Q2, Q3, Q4: BSS138, Package_TO_SOT_SMD:SOT-23, symbol Transistor_FET:BSS138
- removed R10, R11, R12, R13, R14, R15, R16, R17, R18, R19: 10k, Resistor_SMD:R_0402_1005Metric, symbol Device:R_Small
- removed U1: NCP1117-3.3_SOT223, Package_TO_SOT_SMD:SOT-223-3_TabPin2, symbol Regulator_Linear:NCP1117-3.3_SOT223
- removed U2: RP2040, rp2048:RP2040-QFN-56, symbol rp2040:RP2040
- removed U3: ATECC608A-MAHDA, Package_DFN_QFN:DFN-8-1EP_3x2mm_P0.5mm_EP1.3x1.5mm, symbol Security:ATECC608A-MAHDA
- removed U4: W25Q128JVS, Package_SO:SOIC-8_5.23x5.23mm_P1.27mm, symbol Memory_Flash:W25Q128JVS
- added C16, C17: 10u, Capacitor_Tantalum_SMD:CP_EIA-3216-18_Kemet-A, symbol Device:CP1_Small
- added C19, C5, C9: 100n, Capacitor_SMD:C_0402_1005Metric, symbol Device:C_Small
- added D1: B5819W, Diode_SMD:D_SOD-123, symbol Device:D_Schottky_Small
- added J2: SWD, Connector_SWD:20021221-00010C4LF, symbol Connector:Conn_ARM_JTAG_SWD_10
- added J3: GBA-LINK, Connector_GBA:GBA-LINK, symbol Connector_GBA:GBA-LINK
- added J4: GC9A01, Connector_PinHeader_2.54mm:PinHeader_1x08_P2.54mm_Vertical, symbol Connector:Conn_01x08_Female
- added SW1: USB_BOOT, Button_Switch_SMD:SW_Push_1P1T_NO_6x6mm_H9.5mm, symbol Switch:SW_Push
- added U1: ATECC608A-SSHDA, Package_SO:SOIC-8_3.9x4.9mm_P1.27mm, symbol Security:ATECC608A-SSHDA
- added U2: W25Q128JVS, Package_SO:SOIC-8_5.23x5.23mm_P1.27mm, symbol Memory_Flash:W25Q128JVS
- added U3: RP2040, MCU_RaspberryPi_RP2040:RP2040-QFN-56, symbol MCU_RaspberryPi_RP2040:RP2040
- added U4: AMS1117-3.3, Package_TO_SOT_SMD:SOT-223-3_TabPin2, symbol Regulator_Linear:AMS1117-3.3
- added U5: TXS0108EPW, Package_SO:TSSOP-20_4.4x6.5mm_P0.65mm, symbol Logic_LevelTranslator:TXS0108EPW
- C1: value 12p -> 100n; LCSC_PN C387970 -> C1525; Manufacturer Walsin Tech Corp -> (none); Mfg Part # 0402N150G500CT -> (none)
- C10, C12, C13, C14, C18, C8: LCSC_PN C541405 -> C1525; Manufacturer YAGEO -> (none); Mfg Part # CC0402KRX5R5BB104 -> (none)
- C11: value 10u -> 100n; footprint Capacitor_SMD:C_0805_2012Metric -> Capacitor_SMD:C_0402_1005Metric; LCSC_FP 0805 -> 0402; LCSC_PN C408141 -> C1525; Manufacturer Murata Electronics -> (none); Mfg Part # GRM21BR61C106KE15K -> (none)
- C15: value 100n -> 1u; LCSC_PN C541405 -> C52923; Manufacturer YAGEO -> (none); Mfg Part # CC0402KRX5R5BB104 -> (none)
- C2: value 12p -> 22p; LCSC_PN C387970 -> C1555; Manufacturer Walsin Tech Corp -> (none); Mfg Part # 0402N150G500CT -> (none)
- C3: value 100n -> 22p; LCSC_FP 0603 -> 0402; LCSC_PN C167641 -> C1555; Manufacturer Vishay Intertech -> (none); Mfg Part # VJ0603Y104JXACW1BC -> (none)
- C4: LCSC_FP 0603 -> 0402; LCSC_PN C167641 -> C1525; Manufacturer Vishay Intertech -> (none); Mfg Part # VJ0603Y104JXACW1BC -> (none)
- C6: value 2u2 -> 1u; LCSC_PN C193620 -> C52923; Manufacturer FH(Guangdong Fenghua Advanced Tech) -> (none); Mfg Part # 0402X225K6R3NT -> (none)
- C7: value 1u -> 100n; LCSC_PN C193620 -> C1525; Manufacturer FH(Guangdong Fenghua Advanced Tech) -> (none); Mfg Part # 0402X225K6R3NT -> (none)
- H1, H2, H3, H4: footprint MountingHole:MountingHole_3.2mm_M3_Pad_Via -> MountingHole:MountingHole_2.2mm_M2_DIN965_Pad
- J1: value USB_C_Receptacle_USB2.0 -> USB; footprint Connector_USB_C_JLCPCB:TYPE-C-31-M-12 -> Connector_USBC:TYPE-C-31-M-12; LCSC_FP 8.94*7.3mm -> TYPE-C-31_L8.94_W7.3; Manufacturer Korean Hroparts Elec -> (none); Mfg Part # TYPE-C-31-M-12 -> (none)
- R1: LCSC_PN C226166 -> C11702; Manufacturer FH(Guangdong Fenghua Advanced Tech) -> (none); Mfg Part # RC-02W1001FT -> (none)
- R2: value 5.11k -> 1k; LCSC_PN C226166 -> C11702; Manufacturer FH(Guangdong Fenghua Advanced Tech) -> (none); Mfg Part # RC-02W1001FT -> (none)
- R3: value 5.11k -> DNF; LCSC_FP 0402 -> (none); LCSC_PN C226166 -> (none); Manufacturer FH(Guangdong Fenghua Advanced Tech) -> (none); Mfg Part # RC-02W1001FT -> (none)
- R4, R5: value 470 -> 56k; footprint Resistor_SMD:R_0603_1608Metric -> Resistor_SMD:R_0402_1005Metric; LCSC_FP 0603 -> 0402; LCSC_PN C116694 -> C25796; Manufacturer FH(Guangdong Fenghua Advanced Tech) -> (none); Mfg Part # RS-03K4700FT -> (none)
- R6, R7: value 27 -> 10k; LCSC_FP 0603 -> 0402; LCSC_PN C321830 -> C25744; Manufacturer FH(Guangdong Fenghua Advanced Tech) -> (none); Mfg Part # RS-03K27R0FT -> (none)
- R8: value 1k -> 27; LCSC_PN C226166 -> C25100; Manufacturer FH(Guangdong Fenghua Advanced Tech) -> (none); Mfg Part # RC-02W1001FT -> (none)
- R9: value DNF -> 27; LCSC_PN C136582 -> C25100; Manufacturer FH(Guangdong Fenghua Advanced Tech) -> (none); Mfg Part # RC-02000FT -> (none)
- Y1: LCSC_PN C521582 -> C9002; Manufacturer TAITIEN Elec -> (none); Mfg Part # XXHCCLNANF-12.000000MHZ -> (none)
Connections:
- net LED0 is gone; now on net VBUS: R4.1
- net LED1 is gone; now on net VBUS: R5.1
- net MCU_USB_D+ is gone; now on net I2C0_SDA: R6.2
- net MCU_USB_D- is gone; now on net I2C0_SCL: R7.2
- net +1V1: now also C6.1, C7.1, C5.1, U3.23 (DVDD), U3.45 (VREG_VOUT), U3.50 (DVDD); no longer C3.1, C4.1, C6.2
- net +3V3: now also C1.1, C4.1, R3.1, R6.1, R7.1, C17.1, C9.1, D1.2 (A), J4.2 (Pin_2), U1.8 (VCC), U2.8 (VCC), U3.1 (IOVDD), U3.10 (IOVDD), U3.22 (IOVDD), U3.33 (IOVDD), U3.42 (IOVDD), U3.43 (ADC_AVDD), U3.44 (VREG_IN), U3.48 (USB_VDD), U3.49 (IOVDD), U4.2 (VO), U5.10 (OE), U5.2 (VCCA); no longer C7.2, R9.1
- net +5V: now also C19.1, J3.1 (VCC), U5.19 (VCCB)
- net GND: now also C6.2, C7.2, C16.2, C17.2, C19.2, C5.2, C9.2, J2.3 (GND), J2.5 (GND), J2.9 (GNDDetect), J3.6 (GND), J3.7 (SHIELD), J3.8 (SHIELD), J4.1 (Pin_1), SW1.1, U1.4 (GND), U2.4 (GND), U3.19 (TESTEN), U3.57 (GND), U4.1 (GND), U5.11 (GND); no longer C6.1, C7.1, R2.2, R3.1
- net I2C0_SCL: now also U1.6 (SCL), U3.37 (GPIO25)
- net I2C0_SDA: now also U1.5 (SDA), U3.36 (GPIO24)
- net QSPI_SCLK: now also U2.6 (CLK), U3.52 (QSPI_SCLK)
- net QSPI_SD0: now also U2.5 (DI(IO0)), U3.53 (QSPI_SD0)
- net QSPI_SD1: now also U2.2 (DO(IO1)), U3.55 (QSPI_SD1)
- net QSPI_SD2: now also U2.3 (IO2), U3.54 (QSPI_SD2)
- net QSPI_SD3: now also U2.7 (IO3), U3.51 (QSPI_SD3)
- net QSPI_SS: now also R2.1, R3.2, U2.1 (~CS), U3.56 (QSPI_SS); no longer R8.1, R9.2
- net SWCLK: now also J2.4 (SWDCLK/TCK), U3.24 (SWCLK)
- net SWD: now also J2.2 (SWDIO/TMS), U3.25 (SWD)
- net USB_D+: now also R8.2, U3.47 (USB_DP); no longer J1.A6 (D+), J1.B6 (D+), R6.1
- net USB_D-: now also R9.2, U3.46 (USB_DM); no longer J1.A7 (D-), J1.B7 (D-), R7.1
- net VBUS: now also C16.1, D1.1 (K), U4.3 (VI)
- net XIN: now also U3.20 (XIN)
- net XOUT: now also C3.1, Y1.3, U3.21 (XOUT); no longer C1.1, Y1.1
- net ~USB_BOOT: now also R2.2, SW1.2; no longer R8.2
- net at R4.2: now also J1.A5 (CC1)
- net at R5.2: now also J1.B5 (CC2)
- net at C2.1, R1.2: now also Y1.1; no longer Y1.3
- new net GBA_SC: J3.5 (SC), U5.20 (B1)
- new net GBA_SD: J3.4 (SD), U5.16 (B4)
- new net GBA_SI: J3.3 (SI), U5.18 (B2)
- new net GBA_SO: J3.2 (SO), U5.17 (B3)
- new net LCD_BLK: J4.8 (Pin_8), U3.34 (GPIO22)
- new net LCD_CS: J4.7 (Pin_7), U3.28 (GPIO17)
- new net LCD_DC: J4.6 (Pin_6), U3.31 (GPIO20)
- new net LCD_RST: J4.5 (Pin_5), U3.32 (GPIO21)
- new net RUN: U3.26 (RUN)
- new net SPI0_MISO: U3.27 (GPIO16)
- new net SPI0_MOSI: J4.4 (Pin_4), U3.30 (GPIO19)
- new net SPI0_SCLK: J4.3 (Pin_3), U3.29 (GPIO18)
- new net SPI1_CSN: U3.16 (GPIO13), U5.5 (A4)
- new net SPI1_MISO: U3.15 (GPIO12), U5.4 (A3)
- new net SPI1_MOSI: U3.14 (GPIO11), U5.3 (A2)
- new net SPI1_SCLK: U3.13 (GPIO10), U5.1 (A1)
- new net USB_CONN_D+: J1.A6 (D+), J1.B6 (D+), R8.1
- new net USB_CONN_D-: J1.A7 (D-), J1.B7 (D-), R9.1
- no-connect marks 28 -> 31
Other:
- note added: "CL = ((CX1 x CX2) / (CX1 + CX2)) + Cstray\nCX1 = 2(CL - Cstray)"
- note removed: "FLASH"
- note removed: "GBA CONN"
- note removed: "MCU"
- note removed: "NervesKey"
- note removed: "STATUS LEDS\n"
- note removed: "USB+PWR"
